Commit message: tsuchida_moveit

File: denso_run/rikuken_original/tf_publish/urdf/hande_camera.urdf.xacro (robot description, xacro)
@@ -17,7 +17,7 @@
                 <origin xyz="0.0 0.0 0.0" />
                 <mass value="0.63387"/>
-                <inertia ixx = "0.000002" ixy = "0.000000" ixz = "0.000000"
-                    iyx = "0.000000" iyy = "0.000005" iyz = "0.000000"
-                    izx = "0.000000" izy = "0.000000" izz = "0.000006" />
+                <inertia ixx = "0.002" ixy = "0.000000" ixz = "0.000000"
+                    iyx = "0.000000" iyy = "0.005" iyz = "0.000000"
+                    izx = "0.000000" izy = "0.000000" izz = "0.006" />
             </inertial>
             <visual>
@@ -48,7 +48,7 @@
                 <origin xyz="0.0 0.0 0.0" />
                 <mass value="0.03804"/>
-                <inertia ixx = "0.000002" ixy = "0.000000" ixz = "0.000000"
-                        iyx = "0.000000" iyy = "0.000005" iyz = "0.000000"
-                        izx = "0.000000" izy = "0.000000" izz = "0.000006" />
+                <inertia ixx = "0.002" ixy = "0.000000" ixz = "0.000000"
+                        iyx = "0.000000" iyy = "0.005" iyz = "0.000000"
+                        izx = "0.000000" izy = "0.000000" izz = "0.006" />
             </inertial>
             <visual>
@@ -154,7 +154,7 @@
                 <!--origin rpy="0 0 0" xyz="-0.02262 0.00759 0.00738"/-->
                 <mass value="0.03804"/>
-                <inertia ixx = "0.000002" ixy = "0.000000" ixz = "0.000000"
-                        iyx = "0.000000" iyy = "0.000005" iyz = "0.000000"
-                        izx = "0.000000" izy = "0.000000" izz = "0.000006" />
+                <inertia ixx = "0.002" ixy = "0.000000" ixz = "0.000000"
+                        iyx = "0.000000" iyy = "0.005" iyz = "0.000000"
+                        izx = "0.000000" izy = "0.000000" izz = "0.006" />
             </inertial>
             <visual>
@@ -198,6 +198,6 @@
             <forces_angle_tolerance>100</forces_angle_tolerance>
             <update_rate>4</update_rate>
-            <grip_count_threshold>4</grip_count_threshold>
-            <max_grip_count>8</max_grip_count>
+            <grip_count_threshold>2</grip_count_threshold>
+            <max_grip_count>4</max_grip_count>
             <release_tolerance>0.001</release_tolerance>
             <disable_collisions_on_attach>false</disable_collisions_on_attach>

Commit message: tsuchida_next

File: denso_run/rikuken_original/tf_publish/urdf/hande_camera.urdf.xacro (robot description, xacro)
@@ -86,5 +86,5 @@
             </inertial>
             <visual>
-                <material>
+                <material name="green">
                     <color rgba="0.0 1 0.1 1.0"/>
                 </material>
@@ -100,5 +100,5 @@
         </link>
          <gazebo reference="camera_link">
-            <material>Gazebo/Red</material>
+            <material>Gazebo/Green</material>
             <sensor type="camera" name="camera1">
             <update_rate>30.0</update_rate>
