Commit message: fdfd

File: denso_run/rikuken_original/tf_publish/urdf/ur3e_joint_limited_robot.urdf.xacro (robot description, xacro)
@@ -6,4 +6,8 @@
   <!-- ur3e -->
   <xacro:include filename="$(find tf_publish)/urdf/ur3e.urdf.xacro" />
+  <xacro:arg name="ur_x" default="0"/>
+  <xacro:arg name="ur_y" default="0"/>
+  <xacro:arg name="ur_z" default="0"/>
+  <xacro:arg name="ur_yaw" default="1.5"/>
   <!-- arm -->
   <xacro:arg name="kinematics_config" default="$(find tf_publish)/config/ur3e_default.yaml"/>
@@ -23,5 +27,5 @@
     <child link = "base_link" />
     <!-- <origin xyz="-0.5 0.0 1.03" rpy="0.0 0.0 0.0" /> -->
-    <origin xyz="0 0 0" rpy="0.0 0.0 0.0" />
+    <origin xyz="$(arg ur_x) $(arg ur_y) $(arg ur_z)" rpy="0.0 0.0 $(arg ur_yaw)" />
   </joint>
 </robot>
